File: schematics/satellite-outdoor.kicad_sch (KiCad schematic)
At the start: 3 parts, among them U1 LPS22HB, U2 AHT20

Commit message: Revert "Set lps22 i2c address"
This reverts commit cf4319b74ca7d706c925089c18308ba03ea26221.
Connections:
- new net: HTCC-AB02A1. (VIN), U1. (VIN), U2.2 (VDD)
Changed lines of the file:
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@@
-	)
-	(junction
-		(at 88.9 128.27)
-		(diameter 0)
-		(color 0 0 0 0)
 	)
 	(junction
@@
 	(wire
 		(pts
-			(xy 88.9 128.27) (xy 129.54 128.27)
-		)
-		(stroke
-			(width 0)
-			(type default)
-		)
-	)
-	(wire
-		(pts
 			(xy 72.39 46.99) (xy 72.39 64.77)
 		)
@@
 	(wire
 		(pts
-			(xy 88.9 99.06) (xy 88.9 128.27)
-		)
-		(stroke
-			(width 0)
-			(type default)
-		)
-	)
-	(wire
-		(pts
 			(xy 139.7 55.88) (xy 109.22 55.88)
 		)
@@
 	(wire
 		(pts
-			(xy 91.44 105.41) (xy 109.22 105.41)
+			(xy 88.9 105.41) (xy 109.22 105.41)
 		)
 		(stroke
@@
 	(wire
 		(pts
-			(xy 91.44 99.06) (xy 91.44 105.41)
+			(xy 88.9 99.06) (xy 88.9 105.41)
 		)
 		(stroke
@@
 	(wire
 		(pts
-			(xy 83.82 128.27) (xy 88.9 128.27)
-		)
-		(stroke
+			(xy 83.82 128.27) (xy 129.54 128.27)
+		)
+		(stroke

Commit message: Fix LPS22 connection pinout
I2C SDA is SDI pin, not SD0.
Connections:
- new net: HTCC-AB02A1. (VIN), U1. (VIN), U2.2 (VDD)
Changed lines of the file:
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@@
 	(wire
 		(pts
-			(xy 88.9 105.41) (xy 109.22 105.41)
+			(xy 91.44 105.41) (xy 109.22 105.41)
 		)
 		(stroke
@@
 	(wire
 		(pts
-			(xy 88.9 99.06) (xy 88.9 105.41)
+			(xy 91.44 99.06) (xy 91.44 105.41)
 		)
 		(stroke
