File: schematics/satellite-indoor.kicad_sch (KiCad schematic)
At the start: 3 parts, among them IC1 AHT20, U3 SCD40-D-R2

Commit message: Schematics update: use Vext instead of VDD
Vext can be controllled and switched on/off.
Changed lines of the file:
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@@
 	(wire
 		(pts
-			(xy 83.82 68.58) (xy 152.4 68.58)
+			(xy 83.82 68.58) (xy 116.84 68.58)
 		)
 		(stroke
@@
 		(pts
 			(xy 111.76 64.77) (xy 111.76 110.49)
-		)
-		(stroke
-			(width 0)
-			(type default)
-		)
-	)
-	(wire
-		(pts
-			(xy 148.59 85.09) (xy 152.4 85.09)
 		)
 		(stroke
@@
 	(wire
 		(pts
+			(xy 119.38 90.17) (xy 116.84 90.17)
+		)
+		(stroke
+			(width 0)
+			(type default)
+		)
+	)
+	(wire
+		(pts
 			(xy 148.59 87.63) (xy 160.02 87.63)
 		)
@@
 	(wire
 		(pts
-			(xy 152.4 85.09) (xy 152.4 68.58)
-		)
-		(stroke
-			(width 0)
-			(type default)
-		)
-	)
-	(wire
-		(pts
 			(xy 99.06 105.41) (xy 99.06 110.49)
 		)
@@
 		)
 		(stroke
+			(width 0)
+			(type default)
+		)
+	)
+	(wire
+		(pts
+			(xy 116.84 90.17) (xy 116.84 68.58)
+		)
+		(stroke
